File: PottyBoard.kicad_pcb (KiCad board)
At the start: 2 copper layers, 20.3 x 10.2 mm, 12 parts, among them J1 Conn_01x03, J2 Conn_01x03, U1 LMV358

Commit message: PCB layout
Parts:
- added C1: 10n, Capacitor_SMD:C_0402_1005Metric, F.Cu at (151.0, 97.5)
- moved RV2 6.34 mm to (144.0, 97.8)
- moved RV1 5.31 mm to (144.0, 91.2)
- moved R1 3.48 mm to (148.2, 94.0), turned to 0 degrees
- moved R2 2.85 mm to (148.2, 95.2), turned to 180 degrees
- moved R5 1.76 mm to (149.5, 97.5)
- moved C2 1.23 mm to (148.2, 92.8), turned to 180 degrees
- moved J1 0.88 mm to (139.0, 92.0)
- moved J2 0.53 mm to (155.0, 92.0)
- moved R3 0.27 mm to (151.5, 90.5)
- moved R4 0.25 mm to (150.2, 90.5)
- moved R6 0.14 mm to (152.5, 97.5)
Routing:
- net VCC: track 0.00 -> 20.4 mm, vias 0 -> 2
- net Net-(J1-Pin_2): track 0.00 -> 12.1 mm, vias 0 -> 1
- net Net-(U1B-+): track 0.00 -> 9.98 mm, vias 0 -> 2
- net Net-(R2-Pad2): track 0.00 -> 9.17 mm
- net Net-(J2-Pin_2): track 0.00 -> 7.14 mm
- net Net-(U1A-+): track 0.00 -> 5.07 mm
- net Net-(U1A--): track 0.00 -> 4.15 mm
- net Net-(U1B--): track 0.00 -> 3.52 mm
- net Net-(R1-Pad1): track 0.00 -> 2.89 mm
- net GND: vias 0 -> 5
- added copper zone on B.Cu, net GND
- added copper zone on F.Cu, net GND
- added copper zone on In1.Cu, net GND
- added copper zone on In2.Cu, net GND
Other:
- board size 20.3 x 10.2 mm -> 20 x 11 mm
- copper layers 2 -> 4

Commit message: Finish first version
Routing:
- net Net-(R1-Pad1): track 2.89 -> 4.19 mm
- net GND: vias 5 -> 6
Other:
- board text added: "GND"
- board text added: "IN"
- board text added: "OUT"
- board text added: "PottyBoard 0.1"
- board text added: "VCC"
Changed lines of the file:
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@@
       (outputformat 1)
       (mirror false)
-      (drillshape 1)
+      (drillshape 0)
       (scaleselection 1)
-      (outputdirectory "")
+      (outputdirectory "fabrication/")
     )
   )
@@
       (rotate (xyz 0 0 0))
     )
-    (model "${KIPRJMOD}/3dmodels/tc33x-2-xxx.stp"
-      (offset (xyz 0 0 0))
-      (scale (xyz 1 1 1))
-      (rotate (xyz -90 0 90))
-    )
   )
   (footprint "Resistor_SMD:R_0402_1005Metric" (layer "F.Cu")
@@
       (offset (xyz 0 0 0))
       (scale (xyz 1 1 1))
-      (rotate (xyz 90 0 -90))
-    )
-    (model "${KIPRJMOD}/3dmodels/tc33x-2-xxx.stp"
-      (offset (xyz 0 0 0))
-      (scale (xyz 1 1 1))
-      (rotate (xyz -90 0 90))
+      (rotate (xyz 0 0 0))
     )
   )
@@
     (pad "3" thru_hole oval (at 0 5.08) (size 1.7 1.7) (drill 1) (layers "*.Cu" "*.Mask")
       (net 2 "GND") (pinfunction "Pin_3") (pintype "passive"))
-    (model "${KICAD6_3DMODEL_DIR}/Connector_PinHeader_2.54mm.3dshapes/PinHeader_1x03_P2.54mm_Vertical.wrl" hide
+    (model "${KICAD6_3DMODEL_DIR}/Connector_PinHeader_2.54mm.3dshapes/PinHeader_1x03_P2.54mm_Vertical.wrl"
       (offset (xyz 0 0 0))
       (scale (xyz 1 1 1))
@@
     (pad "3" thru_hole oval (at 0 5.08) (size 1.7 1.7) (drill 1) (layers "*.Cu" "*.Mask")
       (net 2 "GND") (pinfunction "Pin_3") (pintype "passive"))
-    (model "${KICAD6_3DMODEL_DIR}/Connector_PinHeader_2.54mm.3dshapes/PinHeader_1x03_P2.54mm_Vertical.wrl" hide
+    (model "${KICAD6_3DMODEL_DIR}/Connector_PinHeader_2.54mm.3dshapes/PinHeader_1x03_P2.54mm_Vertical.wrl"
       (offset (xyz 0 0 0))
       (scale (xyz 1 1 1))
@@
   (gr_rect (start 137 89) (end 157 100)
     (stroke (width 0.1) (type default)) (fill none) (layer "Edge.Cuts"))
+  (gr_text "PottyBoard 0.1" (at 155.6 99.7) (layer "B.SilkS")
+    (effects (font (size 1 1) (thickness 0.15)) (justify left bottom mirror))
+  )
+  (gr_text "OUT" (at 154 95.5) (layer "B.SilkS")
+    (effects (font (size 1.5 1.5) (thickness 0.3) bold) (justify left bottom mirror))
+  )
+  (gr_text "GND" (at 153.9 98) (layer "B.SilkS")
+    (effects (font (size 1.5 1.5) (thickness 0.3) bold) (justify left bottom mirror))
+  )
+  (gr_text "IN" (at 142.9 95.5) (layer "B.SilkS")
+    (effects (font (size 1.5 1.5) (thickness 0.3) bold) (justify left bottom mirror))
+  )
+  (gr_text "VCC" (at 153.9 92.9) (layer "B.SilkS")
+    (effects (font (size 1.5 1.5) (thickness 0.3) bold) (justify left bottom mirror))
+  )
+  (gr_text "GND" (at 144.7 98.1) (layer "B.SilkS")
+    (effects (font (size 1.5 1.5) (thickness 0.3) bold) (justify left bottom mirror))
+  )
+  (gr_text "VCC" (at 144.9 93) (layer "B.SilkS")
+    (effects (font (size 1.5 1.5) (thickness 0.3) bold) (justify left bottom mirror))
+  )
   (dimension (type aligned) (layer "B.Fab")
     (pts (xy 157 100) (xy 157 89))
@@
     (style (thickness 0.1) (arrow_length 1.27) (text_position_mode 0) (extension_height 0.58642) (extension_offset 0.5) keep_text_aligned)
   )
-  (segment (start 141.25 91.2) (end 142.2 90.25) (width 0.25) (layer "F.Cu") (net 1))
   (segment (start 148.73 91.52) (end 148.73 92.75) (width 0.25) (layer "F.Cu") (net 1))
   (segment (start 148.75 91.5) (end 148.73 91.52) (width 0.25) (layer "F.Cu") (net 1))
-  (segment (start 141.25 91.5) (end 141.25 91.2) (width 0.25) (layer "F.Cu") (net 1))
+  (segment (start 141 91.5) (end 141 91.45) (width 0.25) (layer "F.Cu") (net 1))
+  (segment (start 141 91.45) (end 142.2 90.25) (width 0.25) (layer "F.Cu") (net 1))
   (segment (start 148.73 92.75) (end 150.0625 92.75) (width 0.25) (layer "F.Cu") (net 1))
   (segment (start 150.0625 92.75) (end 150.155 92.8425) (width 0.25) (layer "F.Cu") (net 1))
   (via (at 148.75 91.5) (size 0.5) (drill 0.3) (layers "F.Cu" "B.Cu") (net 1))
-  (via (at 141.25 91.5) (size 0.5) (drill 0.3) (layers "F.Cu" "B.Cu") (net 1))
-  (segment (start 148.75 91.5) (end 141.25 91.5) (width 0.25) (layer "B.Cu") (net 1))
-  (segment (start 141.25 91.5) (end 139 91.5) (width 0.25) (layer "B.Cu") (net 1))
-  (segment (start 148.75 91.5) (end 155 91.5) (width 0.25) (layer "B.Cu") (net 1))
+  (via (at 141 91.5) (size 0.5) (drill 0.3) (layers "F.Cu" "B.Cu") (net 1))
+  (segment (start 154.525 91.5) (end 155 91.975) (width 0.25) (layer "B.Cu") (net 1))
+  (segment (start 148.75 91.5) (end 141 91.5) (width 0.25) (layer "B.Cu") (net 1))
+  (segment (start 141 91.5) (end 139.475 91.5) (width 0.25) (layer "B.Cu") (net 1))
+  (segment (start 148.75 91.5) (end 154.525 91.5) (width 0.25) (layer "B.Cu") (net 1))
+  (segment (start 139.475 91.5) (end 139 91.975) (width 0.25) (layer "B.Cu") (net 1))
   (via (at 141.25 92.25) (size 0.5) (drill 0.3) (layers "F.Cu" "B.Cu") (free) (net 2))
   (via (at 141.25 98.75) (size 0.5) (drill 0.3) (layers "F.Cu" "B.Cu") (free) (net 2))
   (via (at 151.75 98) (size 0.5) (drill 0.3) (layers "F.Cu" "B.Cu") (free) (net 2))
   (via (at 147 92.75) (size 0.5) (drill 0.3) (layers "F.Cu" "B.Cu") (free) (net 2))
+  (via (at 152.7 95.1) (size 0.5) (drill 0.3) (layers "F.Cu" "B.Cu") (free) (net 2))
   (via (at 152.25 90) (size 0.5) (drill 0.3) (layers "F.Cu" "B.Cu") (free) (net 2))
   (segment (start 149.5 98.01) (end 148.51 98.01) (width 0.25) (layer "F.Cu") (net 3))
   (segment (start 148.51 98.01) (end 148.5 98) (width 0.25) (layer "F.Cu") (net 3))
   (via (at 148.5 98) (size 0.5) (drill 0.3) (layers "F.Cu" "B.Cu") (net 3))
-  (segment (start 148.5 98) (end 142.96 98) (width 0.25) (layer "B.Cu") (net 3))
-  (segment (start 142.96 98) (end 139 94.04) (width 0.25) (layer "B.Cu") (net 3))
+  (segment (start 139 94.515) (end 142.485 98) (width 0.25) (layer "B.Cu") (net 3))
+  (segment (start 142.485 98) (end 148.5 98) (width 0.25) (layer "B.Cu") (net 3))
   (segment (start 150.805 92.8425) (end 150.805 91.565) (width 0.25) (layer "F.Cu") (net 4))
-  (segment (start 151.340001 94.04) (end 155 94.04) (width 0.25) (layer "F.Cu") (net 4))
-  (segment (start 150.805 93.504999) (end 151.340001 94.04) (width 0.25) (layer "F.Cu") (net 4))
-  (segment (start 150.805 92.8425) (end 150.805 93.504999) (width 0.25) (layer "F.Cu") (net 4))
+  (segment (start 154.18 93.78) (end 151.16085 93.78) (width 0.25) (layer "F.Cu") (net 4))
+  (segment (start 150.805 93.42415) (end 150.805 92.8425) (width 0.25) (layer "F.Cu") (net 4))
+  (segment (start 154.615 94.13) (end 154.53 94.13) (width 0.25) (layer "F.Cu") (net 4))
+  (segment (start 151.16085 93.78) (end 150.805 93.42415) (width 0.25) (layer "F.Cu") (net 4))
+  (segment (start 155 94.515) (end 154.615 94.13) (width 0.25) (layer "F.Cu") (net 4))
+  (segment (start 154.53 94.13) (end 154.18 93.78) (width 0.25) (layer "F.Cu") (net 4))
   (segment (start 150.805 91.565) (end 150.25 91.01) (width 0.25) (layer "F.Cu") (net 4))
+  (segment (start 145.45 92.55) (end 145.45 91.25) (width 0.25) (layer "F.Cu") (net 5))
   (segment (start 146.9 94) (end 145.45 92.55) (width 0.25) (layer "F.Cu") (net 5))
   (segment (start 147.74 94) (end 146.9 94) (width 0.25) (layer "F.Cu") (net 5))
-  (segment (start 150.805 95.1175) (end 150.805 94.455001) (width 0.25) (layer "F.Cu") (net 6))
+  (segment (start 150.805 94.241396) (end 150.563604 94) (width 0.25) (layer "F.Cu") (net 6))
+  (segment (start 150.563604 94) (end 148.76 94) (width 0.25) (layer "F.Cu") (net 6))
+  (segment (start 150.805 95.1175) (end 150.805 94.241396) (width 0.25) (layer "F.Cu") (net 6))
   (segment (start 148.76 95.25) (end 148.76 94) (width 0.25) (layer "F.Cu") (net 6))
-  (segment (start 150.349999 94) (end 148.76 94) (width 0.25) (layer "F.Cu") (net 6))
-  (segment (start 150.805 94.455001) (end 150.349999 94) (width 0.25) (layer "F.Cu") (net 6))
   (segment (start 148.385 95.895) (end 147.74 95.25) (width 0.25) (layer "F.Cu") (net 7))
   (segment (start 143.7 95.25) (end 147.74 95.25) (width 0.25) (layer "F.Cu") (net 7))
@@
   (segment (start 149.5 96.5) (end 152.75 93.25) (width 0.25) (layer "B.Cu") (net 10))
   (zone (net 2) (net_name "GND") (layers "F.Cu" "In1.Cu" "In2.Cu" "B.Cu") (hatch edge 0.5)
-    (connect_pads (clearance 0.3))
+    (connect_pads (clearance 0.2))
     (min_thickness 0.25) (filled_areas_thickness no)
     (fill yes (thermal_gap 0.2) (thermal_bridge_width 0.3))
