File: PottyBoard.kicad_sch (KiCad schematic)
At the start: 13 parts, among them J1 Conn_01x03, J2 Conn_01x03, U1 LMV358

Commit message: Add footprint for filtering capacitor
Parts:
- C1: footprint (none) -> Capacitor_SMD:C_0402_1005Metric
Changed lines of the file:
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@@
       (effects (font (size 1.27 1.27)) (justify left))
     )
-    (property "Footprint" "" (at 97.4852 118.11 0)
+    (property "Footprint" "Capacitor_SMD:C_0402_1005Metric" (at 97.4852 118.11 0)
       (effects (font (size 1.27 1.27)) hide)
     )

Commit message: Finish first version
Changed lines of the file:
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@@
   (junction (at 184.15 96.52) (diameter 0) (color 0 0 0 0)
   )
+  (junction (at 226.06 99.06) (diameter 0) (color 0 0 0 0)
+  )
   (junction (at 101.6 119.38) (diameter 0) (color 0 0 0 0)
   )
+  (junction (at 226.06 93.98) (diameter 0) (color 0 0 0 0)
+  )
   (wire (pts (xy 144.78 182.88) (xy 138.43 182.88))
     (stroke (width 0) (type default))
@@
     (stroke (width 0) (type default))
   )
+  (wire (pts (xy 217.17 99.06) (xy 226.06 99.06))
+    (stroke (width 0) (type default))
+  )
   (wire (pts (xy 130.81 96.52) (xy 152.4 96.52))
     (stroke (width 0) (type default))
@@
   )
   (wire (pts (xy 138.43 171.45) (xy 138.43 167.64))
+    (stroke (width 0) (type default))
+  )
+  (wire (pts (xy 217.17 93.98) (xy 226.06 93.98))
     (stroke (width 0) (type default))
   )
@@
         (path "/403a50c5-5cfe-45f3-869b-807b6e40af74"
           (reference "C1") (unit 1)
+        )
+      )
+    )
+  )
+  (symbol (lib_id "power:PWR_FLAG") (at 217.17 93.98 0) (unit 1)
+    (in_bom yes) (on_board yes) (dnp no) (fields_autoplaced)
+    (property "Reference" "#FLG0101" (at 217.17 92.075 0)
+      (effects (font (size 1.27 1.27)) hide)
+    )
+    (property "Value" "PWR_FLAG" (at 217.17 88.9 0)
+      (effects (font (size 1.27 1.27)))
+    )
+    (property "Footprint" "" (at 217.17 93.98 0)
+      (effects (font (size 1.27 1.27)) hide)
+    )
+    (property "Datasheet" "~" (at 217.17 93.98 0)
+      (effects (font (size 1.27 1.27)) hide)
+    )
+    (pin "1")
+    (instances
+      (project "PottyBoard"
+        (path "/403a50c5-5cfe-45f3-869b-807b6e40af74"
+          (reference "#FLG0101") (unit 1)
         )
       )
@@
         )
       )
+    )
+  )
+  (symbol (lib_id "power:PWR_FLAG") (at 217.17 99.06 180) (unit 1)
+    (in_bom yes) (on_board yes) (dnp no) (fields_autoplaced)
+    (property "Reference" "#FLG0102" (at 217.17 100.965 0)
+      (effects (font (size 1.27 1.27)) hide)
+    )
+    (property "Value" "PWR_FLAG" (at 217.17 104.14 0)
+      (effects (font (size 1.27 1.27)))
+    )
+    (property "Footprint" "" (at 217.17 99.06 0)
+      (effects (font (size 1.27 1.27)) hide)
+    )
+    (property "Datasheet" "~" (at 217.17 99.06 0)
+      (effects (font (size 1.27 1.27)) hide)
+    )
+    (pin "1")
+    (instances
+      (project "PottyBoard"
+        (path "/403a50c5-5cfe-45f3-869b-807b6e40af74"
+          (reference "#FLG0102") (unit 1)
+        )
+      )
